File: Schematic/Complete Schematic V4/Complete Schematic V4.kicad_sch (KiCad schematic)
At the start: 73 parts, among them J1 Conn_Coaxial, J2 USB_A, J3 AudioJack3, U1 Si5351A-B-GT, U2 SN74CBT3253, U3 LT6231, U4 LT6231, U5 LM4562MA, U6 LM4562MA

Commit message: PCB Design
Parts:
- C1, C4: value (none) -> 270p; footprint (none) -> Capacitor_SMD:C_0805_2012Metric
- C10, C11, C12, C26, C27, C9: footprint (none) -> Capacitor_SMD:C_0805_2012Metric
- C13: value (none) -> EEEFK1C100R; footprint (none) -> lmao:CAP_EEEFK1C100R
- C14, C15, C18, C21, C24, C25, C3, C5, C6: value (none) -> 0.1u; footprint (none) -> Capacitor_SMD:C_0805_2012Metric
- C16, C17: value (none) -> 75p; footprint (none) -> Capacitor_SMD:C_0805_2012Metric
- C19, C20, C22, C23: value (none) -> 100p; footprint (none) -> Capacitor_SMD:C_0805_2012Metric
- C2: value (none) -> 560p; footprint (none) -> Capacitor_SMD:C_0805_2012Metric
- C7: value (none) -> 10n; footprint (none) -> Capacitor_SMD:C_0805_2012Metric
- C8: value (none) -> 100n; footprint (none) -> Capacitor_SMD:C_0805_2012Metric
- L1, L2: footprint (none) -> Inductor_SMD:L_0805_2012Metric
- R10, R13, R14, R15, R20, R21: footprint (none) -> Resistor_SMD:R_0805_2012Metric
- R11: value (none) -> 4.64k; footprint (none) -> Resistor_SMD:R_0805_2012Metric
- R12: value (none) -> 52.3k; footprint (none) -> Resistor_SMD:R_0805_2012Metric
- R16, R17: value (none) -> 17.4k; footprint (none) -> Resistor_SMD:R_0805_2012Metric
- R18, R19: value (none) -> 4.7k; footprint (none) -> Resistor_SMD:R_0805_2012Metric
- R2, R8: footprint (none) -> Resistor_SMD:R_2512_6332Metric
- R5, R6: footprint (none) -> Resistor_SMD:R_1206_3216Metric
- TP1: value (none) -> TestPoint; footprint (none) -> TestPoint:TestPoint_THTPad_2.0x2.0mm_Drill1.0mm
- TP10, TP11, TP12, TP2, TP3, TP4, TP5, TP6, TP7, TP8, TP9: footprint (none) -> TestPoint:TestPoint_THTPad_2.0x2.0mm_Drill1.0mm
- Y1: value (none) -> Crystal_GND24_Small; footprint (none) -> Crystal:Crystal_SMD_3225-4Pin_3.2x2.5mm
