File: Schematic/SDRrecV5/Complete Schematic V4.kicad_sch (KiCad schematic)
At the start: 73 parts, among them J1 Conn_Coaxial, U1 Si5351A-B-GT, U2 SN74CBT3253, Y1 Crystal_GND24_Small

Commit message: changes
Parts:
- C13: value (none) -> 8200u; footprint (none) -> Capacitor_THT:CP_Radial_D16.0mm_P7.50mm
- C7: value (none) -> 10n; footprint (none) -> Capacitor_SMD:C_0805_2012Metric
- C8: value (none) -> 100n; footprint (none) -> Capacitor_SMD:C_0805_2012Metric
- J2: value (none) -> SJ1-3525N; footprint (none) -> Audio Jack_Stereo 3:Jack_3.5mm_stereo_TRS_jack
- L2: value (none) -> 360n; footprint (none) -> Inductor_THT:L_Toroid_Vertical_L10.0mm_W5.0mm_P5.08mm
- L3: value (none) -> 750n; footprint (none) -> Inductor_THT:L_Toroid_Vertical_L10.0mm_W5.0mm_P5.08mm
- R1: value (none) -> 1; footprint (none) -> Resistor_SMD:R_0805_2012Metric
- R8, R9: value (none) -> 22k; footprint (none) -> Resistor_SMD:R_0805_2012Metric
- U3: value (none) -> LT6231; footprint (none) -> Package_SO:SOIC-8_3.9x4.9mm_P1.27mm
- U4: value (none) -> LM4562MA; footprint (none) -> Package_SO:SOIC-8_3.9x4.9mm_P1.27mm
Changed lines of the file:
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@@
     (stroke (width 0) (type default) (color 0 0 0 0))
   )
-  (wire (pts (xy 176.53 181.61) (xy 184.15 181.61))
+  (wire (pts (xy 175.26 181.61) (xy 184.15 181.61))
     (stroke (width 0) (type default) (color 0 0 0 0))
   )
@@
       (effects (font (size 1.27 1.27)) hide)
     )
-    (property "Value" "" (id 1) (at 360.68 46.99 0))
+    (property "Value" "PWR_FLAG" (id 1) (at 360.68 46.99 0))
     (property "Footprint" "" (id 2) (at 365.76 43.18 0)
       (effects (font (size 1.27 1.27)) hide)
@@
       (effects (font (size 1.27 1.27)) (justify left))
     )
-    (property "Value" "" (id 1) (at 370.84 52.0699 0)
-      (effects (font (size 1.27 1.27)) (justify left))
-    )
-    (property "Footprint" "" (id 2) (at 372.11 50.8 0)
+    (property "Value" "LM4562MA" (id 1) (at 370.84 52.0699 0)
+      (effects (font (size 1.27 1.27)) (justify left))
+    )
+    (property "Footprint" "Package_SO:SOIC-8_3.9x4.9mm_P1.27mm" (id 2) (at 372.11 50.8 0)
       (effects (font (size 1.27 1.27)) hide)
     )
@@
       (effects (font (size 1.27 1.27)) (justify left))
     )
-    (property "Value" "" (id 1) (at 227.33 185.8009 0)
-      (effects (font (size 1.27 1.27)) (justify left))
-    )
-    (property "Footprint" "" (id 2) (at 224.4852 189.23 0)
+    (property "Value" "8200u" (id 1) (at 227.33 185.8009 0)
+      (effects (font (size 1.27 1.27)) (justify left))
+    )
+    (property "Footprint" "Capacitor_THT:CP_Radial_D16.0mm_P7.50mm" (id 2) (at 224.4852 189.23 0)
       (effects (font (size 1.27 1.27)) hide)
     )
@@
     (in_bom yes) (on_board yes)
     (property "Reference" "R9" (id 0) (at 255.27 111.76 90))
-    (property "Value" "" (id 1) (at 255.27 114.3 90))
-    (property "Footprint" "" (id 2) (at 250.19 117.348 90)
+    (property "Value" "22k" (id 1) (at 255.27 114.3 90))
+    (property "Footprint" "Resistor_SMD:R_0805_2012Metric" (id 2) (at 250.19 117.348 90)
       (effects (font (size 1.27 1.27)) hide)
     )
@@
       (effects (font (size 1.27 1.27)) (justify left))
     )
-    (property "Value" "" (id 1) (at 267.97 38.0999 0)
-      (effects (font (size 1.27 1.27)) (justify left))
-    )
-    (property "Footprint" "" (id 2) (at 269.24 36.83 0)
+    (property "Value" "LT6231" (id 1) (at 267.97 38.0999 0)
+      (effects (font (size 1.27 1.27)) (justify left))
+    )
+    (property "Footprint" "Package_SO:SOIC-8_3.9x4.9mm_P1.27mm" (id 2) (at 269.24 36.83 0)
       (effects (font (size 1.27 1.27)) hide)
     )
@@
     (in_bom yes) (on_board yes) (fields_autoplaced)
     (property "Reference" "L3" (id 0) (at 114.3 73.66 90))
-    (property "Value" "" (id 1) (at 114.3 76.2 90))
-    (property "Footprint" "" (id 2) (at 114.3 80.01 0)
+    (property "Value" "750n" (id 1) (at 114.3 76.2 90))
+    (property "Footprint" "Inductor_THT:L_Toroid_Vertical_L10.0mm_W5.0mm_P5.08mm" (id 2) (at 114.3 80.01 0)
       (effects (font (size 1.27 1.27)) hide)
     )
@@
     (in_bom yes) (on_board yes) (fields_autoplaced)
     (property "Reference" "U4" (id 0) (at 326.39 68.58 0))
-    (property "Value" "" (id 1) (at 326.39 71.12 0))
-    (property "Footprint" "" (id 2) (at 326.39 78.74 0)
+    (property "Value" "LM4562MA" (id 1) (at 326.39 71.12 0))
+    (property "Footprint" "Package_SO:SOIC-8_3.9x4.9mm_P1.27mm" (id 2) (at 326.39 78.74 0)
       (effects (font (size 1.27 1.27)) hide)
     )
@@
       (effects (font (size 1.27 1.27)) (justify left))
     )
-    (property "Value" "" (id 1) (at 201.93 186.6899 0)
-      (effects (font (size 1.27 1.27)) (justify left))
-    )
-    (property "Footprint" "" (id 2) (at 199.0852 189.23 0)
+    (property "Value" "10n" (id 1) (at 201.93 186.6899 0)
+      (effects (font (size 1.27 1.27)) (justify left))
+    )
+    (property "Footprint" "Capacitor_SMD:C_0805_2012Metric" (id 2) (at 199.0852 189.23 0)
       (effects (font (size 1.27 1.27)) hide)
     )
@@
       (effects (font (size 1.27 1.27)) (justify left))
     )
-    (property "Value" "" (id 1) (at 213.36 186.6899 0)
-      (effects (font (size 1.27 1.27)) (justify left))
-    )
-    (property "Footprint" "" (id 2) (at 210.5152 189.23 0)
+    (property "Value" "100n" (id 1) (at 213.36 186.6899 0)
+      (effects (font (size 1.27 1.27)) (justify left))
+    )
+    (property "Footprint" "Capacitor_SMD:C_0805_2012Metric" (id 2) (at 210.5152 189.23 0)
       (effects (font (size 1.27 1.27)) hide)
     )
@@
     (in_bom yes) (on_board yes) (fields_autoplaced)
     (property "Reference" "U4" (id 0) (at 326.39 83.82 0))
-    (property "Value" "" (id 1) (at 326.39 86.36 0))
-    (property "Footprint" "" (id 2) (at 326.39 93.98 0)
+    (property "Value" "LM4562MA" (id 1) (at 326.39 86.36 0))
+    (property "Footprint" "Package_SO:SOIC-8_3.9x4.9mm_P1.27mm" (id 2) (at 326.39 93.98 0)
       (effects (font (size 1.27 1.27)) hide)
     )
@@
     (in_bom yes) (on_board yes)
     (property "Reference" "R8" (id 0) (at 254 74.93 90))
-    (property "Value" "" (id 1) (at 255.27 77.47 90))
-    (property "Footprint" "" (id 2) (at 250.19 81.788 90)
+    (property "Value" "22k" (id 1) (at 255.27 77.47 90))
+    (property "Footprint" "Resistor_SMD:R_0805_2012Metric" (id 2) (at 250.19 81.788 90)
       (effects (font (size 1.27 1.27)) hide)
     )
@@
       (effects (font (size 1.27 1.27)) (justify left))
     )
-    (property "Value" "" (id 1) (at 93.98 88.8999 0)
-      (effects (font (size 1.27 1.27)) (justify left))
-    )
-    (property "Footprint" "" (id 2) (at 92.71 87.63 0)
+    (property "Value" "360n" (id 1) (at 93.98 88.8999 0)
+      (effects (font (size 1.27 1.27)) (justify left))
+    )
+    (property "Footprint" "Inductor_THT:L_Toroid_Vertical_L10.0mm_W5.0mm_P5.08mm" (id 2) (at 92.71 87.63 0)
       (effects (font (size 1.27 1.27)) hide)
     )
@@
     (in_bom yes) (on_board yes) (fields_autoplaced)
     (property "Reference" "U3" (id 0) (at 250.19 55.88 0))
-    (property "Value" "" (id 1) (at 250.19 58.42 0))
-    (property "Footprint" "" (id 2) (at 250.19 66.04 0)
+    (property "Value" "LT6231" (id 1) (at 250.19 58.42 0))
+    (property "Footprint" "Package_SO:SOIC-8_3.9x4.9mm_P1.27mm" (id 2) (at 250.19 66.04 0)
       (effects (font (size 1.27 1.27)) hide)
     )
@@
     (pin "1")
   )
-  (symbol (lib_id "power:+5V") (at 176.53 181.61 0) (unit 1)
-    (in_bom yes) (on_board yes) (fields_autoplaced)
-    (property "Reference" "#PWR05" (id 0) (at 176.53 185.42 0)
-      (effects (font (size 1.27 1.27)) hide)
-    )
-    (property "Value" "+5V" (id 1) (at 176.53 176.53 0))
-    (property "Footprint" "" (id 2) (at 176.53 181.61 0)
-      (effects (font (size 1.27 1.27)) hide)
-    )
-    (property "Datasheet" "" (id 3) (at 176.53 181.61 0)
+  (symbol (lib_id "power:+5V") (at 175.26 181.61 0) (unit 1)
+    (in_bom yes) (on_board yes) (fields_autoplaced)
+    (property "Reference" "#PWR05" (id 0) (at 175.26 185.42 0)
+      (effects (font (size 1.27 1.27)) hide)
+    )
+    (property "Value" "+5V" (id 1) (at 175.26 176.53 0))
+    (property "Footprint" "" (id 2) (at 175.26 181.61 0)
+      (effects (font (size 1.27 1.27)) hide)
+    )
+    (property "Datasheet" "" (id 3) (at 175.26 181.61 0)
       (effects (font (size 1.27 1.27)) hide)
     )
@@
     (in_bom yes) (on_board yes) (fields_autoplaced)
     (property "Reference" "R1" (id 0) (at 187.96 175.26 90))
-    (property "Value" "" (id 1) (at 187.96 177.8 90))
-    (property "Footprint" "" (id 2) (at 187.96 183.388 90)
+    (property "Value" "1" (id 1) (at 187.96 177.8 90))
+    (property "Footprint" "Resistor_SMD:R_0805_2012Metric" (id 2) (at 187.96 183.388 90)
       (effects (font (size 1.27 1.27)) hide)
     )
@@
     (in_bom yes) (on_board yes) (fields_autoplaced)
     (property "Reference" "U3" (id 0) (at 250.19 91.44 0))
-    (property "Value" "" (id 1) (at 250.19 93.98 0))
-    (property "Footprint" "" (id 2) (at 250.19 101.6 0)
+    (property "Value" "LT6231" (id 1) (at 250.19 93.98 0))
+    (property "Footprint" "Package_SO:SOIC-8_3.9x4.9mm_P1.27mm" (id 2) (at 250.19 101.6 0)
       (effects (font (size 1.27 1.27)) hide)
     )
@@
       (effects (font (size 1.27 1.27)) (justify right))
     )
-    (property "Value" "" (id 1) (at 391.16 86.3599 0)
-      (effects (font (size 1.27 1.27)) (justify right))
-    )
-    (property "Footprint" "" (id 2) (at 379.73 85.09 0)
+    (property "Value" "SJ1-3525N" (id 1) (at 391.16 86.3599 0)
+      (effects (font (size 1.27 1.27)) (justify right))
+    )
+    (property "Footprint" "Audio Jack_Stereo 3:Jack_3.5mm_stereo_TRS_jack" (id 2) (at 379.73 85.09 0)
       (effects (font (size 1.27 1.27)) (justify left bottom) hide)
     )
