File: Schematic/SDRrecV5/Complete Schematic V4.kicad_sch (KiCad schematic)
At the start: 61 parts, among them J1 Conn_Coaxial, U4 LT6231, U6 LM4562MA, Y1 Crystal

Commit message: Final Schematic and PCB
Parts:
- removed C13: (no value), symbol EEEFK1C100R:EEEFK1C100R
- removed C25: (no value), symbol Device:C
- removed J2: (no value), symbol Connector:USB_A
- removed J3: (no value), symbol Connector:AudioJack3
- removed U3, U5: (no value), symbol pspice:OPAMP
- removed U4: LT6231, Package_SO:SOIC-8_3.9x4.9mm_P1.27mm, symbol pspice:OPAMP
- removed U6: LM4562MA, Package_SO:SOIC-8_3.9x4.9mm_P1.27mm, symbol pspice:OPAMP
- removed Y1: Crystal, symbol Device:Crystal
- added C13: (no value), symbol Device:C_Polarized
- added J2: (no value), symbol SJ1-3525N:SJ1-3525N
- added R1: (no value), symbol Device:R
- added TP1, TP10, TP11, TP12, TP13, TP14, TP15, TP2, TP3, TP4, TP5, TP6, TP7, TP8, TP9: TestPoint, TestPoint:TestPoint_THTPad_2.0x2.0mm_Drill1.0mm, symbol Connector:TestPoint
- added U3, U4: (no value), symbol lt6231:LT6231
- added Y1: Crystal_GND24_Small, Crystal:Crystal_SMD_3225-4Pin_3.2x2.5mm, symbol Device:Crystal_GND24_Small
- A1: value (none) -> Arduino_Nano_v3.x; footprint (none) -> Module:Arduino_Nano
- C1: value (none) -> 270p; footprint (none) -> Capacitor_SMD:C_0805_2012Metric
- C10, C11, C12, C9: value (none) -> 5n; footprint (none) -> Capacitor_SMD:C_0805_2012Metric
- C14, C15, C18, C21, C24, C3, C5, C6: value (none) -> 0.1u; footprint (none) -> Capacitor_SMD:C_0805_2012Metric
- C16, C17: value (none) -> 75p; footprint (none) -> Capacitor_SMD:C_0805_2012Metric
- C19, C20, C22, C23: value (none) -> 100p; footprint (none) -> Capacitor_SMD:C_0805_2012Metric
- C2: value (none) -> 560p; footprint (none) -> Capacitor_SMD:C_0805_2012Metric
- C26, C27: value (none) -> 10u; footprint (none) -> Capacitor_SMD:C_0805_2012Metric
- L1: value 750n -> (none); footprint Inductor_SMD:L_0805_2012Metric -> (none)
- L2: value 360n -> (none); footprint Inductor_SMD:L_0805_2012Metric -> (none)
- R10, R11: value (none) -> 4.64k; footprint (none) -> Resistor_SMD:R_0805_2012Metric
- R12, R13: value (none) -> 52.3k; footprint (none) -> Resistor_SMD:R_0805_2012Metric
- R14, R15: value (none) -> 2.49k; footprint (none) -> Resistor_SMD:R_0805_2012Metric
- R16, R17: value (none) -> 17.4k; footprint (none) -> Resistor_SMD:R_0805_2012Metric
- R18, R19: value (none) -> 4.7k; footprint (none) -> Resistor_SMD:R_0805_2012Metric
- R20, R21: value (none) -> 100; footprint (none) -> Resistor_SMD:R_0805_2012Metric
- R4, R5, R6, R7: value (none) -> 200; footprint (none) -> Resistor_SMD:R_1206_3216Metric
- U1: value (none) -> Si5351A-B-GT; footprint (none) -> Package_SO:MSOP-10_3x3mm_P0.5mm
- U2: value (none) -> SN74CBT3253; footprint (none) -> Package_SO:SOIC-16_3.9x9.9mm_P1.27mm
Connections:
- net +5V: now also R1.1
- net Filtered 5V: now also C13.1, R1.2, U3.8 (V+), U4.8 (V+)
- net GND: now also C13.2, J2.1, U3.4 (V-), U4.4 (V-), Y1.2, Y1.4
- net at C1.2, J1.2 (Ext): now also TP1.1
- net at R20.1: now also J2.3
- net at C26.1, R20.2: now also TP11.1
- net at C17.2, R7.2, R9.1: now also U3.6 (-)
- net at C17.1, R11.2, R9.2: now also TP8.1, U3.7
- net at R4.2: now also U3.3 (+)
- net at C16.2, R5.2, R8.1: now also U3.2 (-)
- net at C16.1, R10.1, R8.2: now also TP7.1, U3.1
- net at C10.2, R5.1, U2.11 (2B2)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: now also TP4.1
- net at R14.1, R16.1: now also U4.3 (+)
- net at C19.2, C26.2, R16.2: now also U4.1
- net at C12.2, R7.1, U2.13 (2B4)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: now also TP6.1
- net at C11.1, R6.1, U2.12 (2B3)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: now also TP5.1
- net at C22.1, R12.1: now also U4.2 (-)
- net at L3.2, R2.2, R3.1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: now also TP2.1
- net at R6.2: now also U3.5 (+)
- net at C9.1, R4.1, U2.10 (2B1)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: now also TP3.1
- net at U1.10 (CLK0), U2.14 (S0): now also TP14.1
- net at U1.9 (CLK1), U2.2 (S1): now also TP15.1
- net at C23.2, R13.1: now also U4.5 (+)
- net at R15.2, R17.2: now also U4.6 (-)
- net at C20.2, C27.2, R17.1: now also U4.7
- net at C19.1, R10.2, R12.2: now also TP9.1
- net at C20.1, R11.1, R13.2: now also TP10.1
- net at R21.1: now also J2.2
- net at C27.1, R21.2: now also TP12.1
- net at U1.3 (XB): now also Y1.1
- net at U1.2 (XA): now also Y1.3
- net at U1.6 (CLK2): now also TP13.1
- no-connect marks 28 -> 26
Other:
- moved on the sheet: C14, C15, C7, C8

Commit message: trying to update christian v3
Parts:
- C13: value (none) -> 8200u; footprint (none) -> Capacitor_THT:CP_Radial_D16.0mm_P7.50mm
- C7: value (none) -> 10n; footprint (none) -> Capacitor_SMD:C_0805_2012Metric
- C8: value (none) -> 100n; footprint (none) -> Capacitor_SMD:C_0805_2012Metric
- J2: value (none) -> SJ1-3525N; footprint (none) -> Audio Jack_Stereo 3:Jack_3.5mm_stereo_TRS_jack
- L1, L3: value (none) -> 750n; footprint (none) -> Inductor_THT:L_Toroid_Vertical_L10.0mm_W5.0mm_P5.08mm
- L2: value (none) -> 360n; footprint (none) -> Inductor_THT:L_Toroid_Vertical_L10.0mm_W5.0mm_P5.08mm
- R1: value (none) -> 1; footprint (none) -> Resistor_SMD:R_0805_2012Metric
- R8, R9: value (none) -> 22k; footprint (none) -> Resistor_SMD:R_0805_2012Metric
- U3: value (none) -> LT6231; footprint (none) -> Package_SO:SOIC-8_3.9x4.9mm_P1.27mm
- U4: value (none) -> LM4562MA; footprint (none) -> Package_SO:SOIC-8_3.9x4.9mm_P1.27mm
Changed lines of the file:
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@@
     (stroke (width 0) (type default) (color 0 0 0 0))
   )
-  (wire (pts (xy 176.53 181.61) (xy 184.15 181.61))
+  (wire (pts (xy 175.26 181.61) (xy 184.15 181.61))
     (stroke (width 0) (type default) (color 0 0 0 0))
   )
@@
       (effects (font (size 1.27 1.27)) hide)
     )
-    (property "Value" "" (id 1) (at 360.68 46.99 0))
+    (property "Value" "PWR_FLAG" (id 1) (at 360.68 46.99 0))
     (property "Footprint" "" (id 2) (at 365.76 43.18 0)
       (effects (font (size 1.27 1.27)) hide)
@@
       (effects (font (size 1.27 1.27)) (justify left))
     )
-    (property "Value" "" (id 1) (at 370.84 52.0699 0)
-      (effects (font (size 1.27 1.27)) (justify left))
-    )
-    (property "Footprint" "" (id 2) (at 372.11 50.8 0)
+    (property "Value" "LM4562MA" (id 1) (at 370.84 52.0699 0)
+      (effects (font (size 1.27 1.27)) (justify left))
+    )
+    (property "Footprint" "Package_SO:SOIC-8_3.9x4.9mm_P1.27mm" (id 2) (at 372.11 50.8 0)
       (effects (font (size 1.27 1.27)) hide)
     )
@@
       (effects (font (size 1.27 1.27)) (justify left))
     )
-    (property "Value" "" (id 1) (at 227.33 185.8009 0)
-      (effects (font (size 1.27 1.27)) (justify left))
-    )
-    (property "Footprint" "" (id 2) (at 224.4852 189.23 0)
+    (property "Value" "8200u" (id 1) (at 227.33 185.8009 0)
+      (effects (font (size 1.27 1.27)) (justify left))
+    )
+    (property "Footprint" "Capacitor_THT:CP_Radial_D16.0mm_P7.50mm" (id 2) (at 224.4852 189.23 0)
       (effects (font (size 1.27 1.27)) hide)
     )
@@
     (in_bom yes) (on_board yes)
     (property "Reference" "R9" (id 0) (at 255.27 111.76 90))
-    (property "Value" "" (id 1) (at 255.27 114.3 90))
-    (property "Footprint" "" (id 2) (at 250.19 117.348 90)
+    (property "Value" "22k" (id 1) (at 255.27 114.3 90))
+    (property "Footprint" "Resistor_SMD:R_0805_2012Metric" (id 2) (at 250.19 117.348 90)
       (effects (font (size 1.27 1.27)) hide)
     )
@@
       (effects (font (size 1.27 1.27)) (justify left))
     )
-    (property "Value" "" (id 1) (at 267.97 38.0999 0)
-      (effects (font (size 1.27 1.27)) (justify left))
-    )
-    (property "Footprint" "" (id 2) (at 269.24 36.83 0)
+    (property "Value" "LT6231" (id 1) (at 267.97 38.0999 0)
+      (effects (font (size 1.27 1.27)) (justify left))
+    )
+    (property "Footprint" "Package_SO:SOIC-8_3.9x4.9mm_P1.27mm" (id 2) (at 269.24 36.83 0)
       (effects (font (size 1.27 1.27)) hide)
     )
@@
     (in_bom yes) (on_board yes) (fields_autoplaced)
     (property "Reference" "L3" (id 0) (at 114.3 73.66 90))
-    (property "Value" "" (id 1) (at 114.3 76.2 90))
-    (property "Footprint" "" (id 2) (at 114.3 80.01 0)
+    (property "Value" "750n" (id 1) (at 114.3 76.2 90))
+    (property "Footprint" "Inductor_THT:L_Toroid_Vertical_L10.0mm_W5.0mm_P5.08mm" (id 2) (at 114.3 80.01 0)
       (effects (font (size 1.27 1.27)) hide)
     )
@@
     (in_bom yes) (on_board yes) (fields_autoplaced)
     (property "Reference" "U4" (id 0) (at 326.39 68.58 0))
-    (property "Value" "" (id 1) (at 326.39 71.12 0))
-    (property "Footprint" "" (id 2) (at 326.39 78.74 0)
+    (property "Value" "LM4562MA" (id 1) (at 326.39 71.12 0))
+    (property "Footprint" "Package_SO:SOIC-8_3.9x4.9mm_P1.27mm" (id 2) (at 326.39 78.74 0)
       (effects (font (size 1.27 1.27)) hide)
     )
@@
       (effects (font (size 1.27 1.27)) (justify left))
     )
-    (property "Value" "" (id 1) (at 201.93 186.6899 0)
-      (effects (font (size 1.27 1.27)) (justify left))
-    )
-    (property "Footprint" "" (id 2) (at 199.0852 189.23 0)
+    (property "Value" "10n" (id 1) (at 201.93 186.6899 0)
+      (effects (font (size 1.27 1.27)) (justify left))
+    )
+    (property "Footprint" "Capacitor_SMD:C_0805_2012Metric" (id 2) (at 199.0852 189.23 0)
       (effects (font (size 1.27 1.27)) hide)
     )
@@
     (in_bom yes) (on_board yes) (fields_autoplaced)
     (property "Reference" "L1" (id 0) (at 74.93 73.66 90))
-    (property "Value" "" (id 1) (at 74.93 76.2 90))
-    (property "Footprint" "" (id 2) (at 74.93 80.01 0)
+    (property "Value" "750n" (id 1) (at 74.93 76.2 90))
+    (property "Footprint" "Inductor_THT:L_Toroid_Vertical_L10.0mm_W5.0mm_P5.08mm" (id 2) (at 74.93 80.01 0)
       (effects (font (size 1.27 1.27)) hide)
     )
@@
       (effects (font (size 1.27 1.27)) (justify left))
     )
-    (property "Value" "" (id 1) (at 213.36 186.6899 0)
-      (effects (font (size 1.27 1.27)) (justify left))
-    )
-    (property "Footprint" "" (id 2) (at 210.5152 189.23 0)
+    (property "Value" "100n" (id 1) (at 213.36 186.6899 0)
+      (effects (font (size 1.27 1.27)) (justify left))
+    )
+    (property "Footprint" "Capacitor_SMD:C_0805_2012Metric" (id 2) (at 210.5152 189.23 0)
       (effects (font (size 1.27 1.27)) hide)
     )
@@
     (in_bom yes) (on_board yes) (fields_autoplaced)
     (property "Reference" "U4" (id 0) (at 326.39 83.82 0))
-    (property "Value" "" (id 1) (at 326.39 86.36 0))
-    (property "Footprint" "" (id 2) (at 326.39 93.98 0)
+    (property "Value" "LM4562MA" (id 1) (at 326.39 86.36 0))
+    (property "Footprint" "Package_SO:SOIC-8_3.9x4.9mm_P1.27mm" (id 2) (at 326.39 93.98 0)
       (effects (font (size 1.27 1.27)) hide)
     )
@@
     (in_bom yes) (on_board yes)
     (property "Reference" "R8" (id 0) (at 254 74.93 90))
-    (property "Value" "" (id 1) (at 255.27 77.47 90))
-    (property "Footprint" "" (id 2) (at 250.19 81.788 90)
+    (property "Value" "22k" (id 1) (at 255.27 77.47 90))
+    (property "Footprint" "Resistor_SMD:R_0805_2012Metric" (id 2) (at 250.19 81.788 90)
       (effects (font (size 1.27 1.27)) hide)
     )
@@
       (effects (font (size 1.27 1.27)) (justify left))
     )
-    (property "Value" "" (id 1) (at 93.98 88.8999 0)
-      (effects (font (size 1.27 1.27)) (justify left))
-    )
-    (property "Footprint" "" (id 2) (at 92.71 87.63 0)
+    (property "Value" "360n" (id 1) (at 93.98 88.8999 0)
+      (effects (font (size 1.27 1.27)) (justify left))
+    )
+    (property "Footprint" "Inductor_THT:L_Toroid_Vertical_L10.0mm_W5.0mm_P5.08mm" (id 2) (at 92.71 87.63 0)
       (effects (font (size 1.27 1.27)) hide)
     )
@@
     (in_bom yes) (on_board yes) (fields_autoplaced)
     (property "Reference" "U3" (id 0) (at 250.19 55.88 0))
-    (property "Value" "" (id 1) (at 250.19 58.42 0))
-    (property "Footprint" "" (id 2) (at 250.19 66.04 0)
+    (property "Value" "LT6231" (id 1) (at 250.19 58.42 0))
+    (property "Footprint" "Package_SO:SOIC-8_3.9x4.9mm_P1.27mm" (id 2) (at 250.19 66.04 0)
       (effects (font (size 1.27 1.27)) hide)
     )
@@
     (pin "1")
   )
-  (symbol (lib_id "power:+5V") (at 176.53 181.61 0) (unit 1)
-    (in_bom yes) (on_board yes) (fields_autoplaced)
-    (property "Reference" "#PWR05" (id 0) (at 176.53 185.42 0)
-      (effects (font (size 1.27 1.27)) hide)
-    )
-    (property "Value" "+5V" (id 1) (at 176.53 176.53 0))
-    (property "Footprint" "" (id 2) (at 176.53 181.61 0)
-      (effects (font (size 1.27 1.27)) hide)
-    )
-    (property "Datasheet" "" (id 3) (at 176.53 181.61 0)
+  (symbol (lib_id "power:+5V") (at 175.26 181.61 0) (unit 1)
+    (in_bom yes) (on_board yes) (fields_autoplaced)
+    (property "Reference" "#PWR05" (id 0) (at 175.26 185.42 0)
+      (effects (font (size 1.27 1.27)) hide)
+    )
+    (property "Value" "+5V" (id 1) (at 175.26 176.53 0))
+    (property "Footprint" "" (id 2) (at 175.26 181.61 0)
+      (effects (font (size 1.27 1.27)) hide)
+    )
+    (property "Datasheet" "" (id 3) (at 175.26 181.61 0)
       (effects (font (size 1.27 1.27)) hide)
     )
@@
     (in_bom yes) (on_board yes) (fields_autoplaced)
     (property "Reference" "R1" (id 0) (at 187.96 175.26 90))
-    (property "Value" "" (id 1) (at 187.96 177.8 90))
-    (property "Footprint" "" (id 2) (at 187.96 183.388 90)
+    (property "Value" "1" (id 1) (at 187.96 177.8 90))
+    (property "Footprint" "Resistor_SMD:R_0805_2012Metric" (id 2) (at 187.96 183.388 90)
       (effects (font (size 1.27 1.27)) hide)
     )
@@
     (in_bom yes) (on_board yes) (fields_autoplaced)
     (property "Reference" "U3" (id 0) (at 250.19 91.44 0))
-    (property "Value" "" (id 1) (at 250.19 93.98 0))
-    (property "Footprint" "" (id 2) (at 250.19 101.6 0)
+    (property "Value" "LT6231" (id 1) (at 250.19 93.98 0))
+    (property "Footprint" "Package_SO:SOIC-8_3.9x4.9mm_P1.27mm" (id 2) (at 250.19 101.6 0)
       (effects (font (size 1.27 1.27)) hide)
     )
@@
       (effects (font (size 1.27 1.27)) (justify right))
     )
-    (property "Value" "" (id 1) (at 391.16 86.3599 0)
-      (effects (font (size 1.27 1.27)) (justify right))
-    )
-    (property "Footprint" "" (id 2) (at 379.73 85.09 0)
+    (property "Value" "SJ1-3525N" (id 1) (at 391.16 86.3599 0)
+      (effects (font (size 1.27 1.27)) (justify right))
+    )
+    (property "Footprint" "Audio Jack_Stereo 3:Jack_3.5mm_stereo_TRS_jack" (id 2) (at 379.73 85.09 0)
       (effects (font (size 1.27 1.27)) (justify left bottom) hide)
     )

Commit message: updated values
Parts:
- C10, C11, C12, C9: value 5n -> (none); footprint Capacitor_SMD:C_0805_2012Metric -> (none)
- R8, R9: value 22k -> (none); footprint Resistor_SMD:R_0805_2012Metric -> (none)
Changed lines of the file:
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@@
     (in_bom yes) (on_board yes)
     (property "Reference" "R9" (id 0) (at 255.27 111.76 90))
-    (property "Value" "22k" (id 1) (at 255.27 114.3 90))
-    (property "Footprint" "Resistor_SMD:R_0805_2012Metric" (id 2) (at 250.19 117.348 90)
-      (effects (font (size 1.27 1.27)) hide)
-    )
-    (property "Datasheet" "https://www.meritekusa.com/wp-content/uploads/2018/06/Standard-Chip-Resistor-CR-Series.pdf" (id 3) (at 250.19 115.57 0)
+    (property "Value" "" (id 1) (at 255.27 114.3 90))
+    (property "Footprint" "" (id 2) (at 250.19 117.348 90)
+      (effects (font (size 1.27 1.27)) hide)
+    )
+    (property "Datasheet" "https://www.te.com/commerce/DocumentDelivery/DDEController?Action=srchrtrv&DocNm=1773204&DocType=DS&DocLang=English" (id 3) (at 250.19 115.57 0)
       (effects (font (size 1.27 1.27)) hide)
     )
@@
       (effects (font (size 1.27 1.27)) (justify right))
     )
-    (property "Value" "5n" (id 1) (at 217.17 73.6599 0)
-      (effects (font (size 1.27 1.27)) (justify right))
-    )
-    (property "Footprint" "Capacitor_SMD:C_0805_2012Metric" (id 2) (at 212.3948 68.58 0)
-      (effects (font (size 1.27 1.27)) hide)
-    )
-    (property "Datasheet" "https://datasheets.kyocera-avx.com/X7RDielectric.pdf" (id 3) (at 213.36 72.39 0)
+    (property "Value" "" (id 1) (at 217.17 73.6599 0)
+      (effects (font (size 1.27 1.27)) (justify right))
+    )
+    (property "Footprint" "" (id 2) (at 212.3948 68.58 0)
+      (effects (font (size 1.27 1.27)) hide)
+    )
+    (property "Datasheet" "https://search.murata.co.jp/Ceramy/image/img/A01X/G101/ENG/GRM2195C1H512JA01-01.pdf" (id 3) (at 213.36 72.39 0)
       (effects (font (size 1.27 1.27)) hide)
     )
@@
       (effects (font (size 1.27 1.27)) (justify right))
     )
-    (property "Value" "5n" (id 1) (at 217.17 96.5199 0)
-      (effects (font (size 1.27 1.27)) (justify right))
-    )
-    (property "Footprint" "Capacitor_SMD:C_0805_2012Metric" (id 2) (at 212.3948 91.44 0)
-      (effects (font (size 1.27 1.27)) hide)
-    )
-    (property "Datasheet" "https://datasheets.kyocera-avx.com/X7RDielectric.pdf" (id 3) (at 213.36 95.25 0)
+    (property "Value" "" (id 1) (at 217.17 96.5199 0)
+      (effects (font (size 1.27 1.27)) (justify right))
+    )
+    (property "Footprint" "" (id 2) (at 212.3948 91.44 0)
+      (effects (font (size 1.27 1.27)) hide)
+    )
+    (property "Datasheet" "https://search.murata.co.jp/Ceramy/image/img/A01X/G101/ENG/GRM2195C1H512JA01-01.pdf" (id 3) (at 213.36 95.25 0)
       (effects (font (size 1.27 1.27)) hide)
     )
@@
       (effects (font (size 1.27 1.27)) (justify right))
     )
-    (property "Value" "5n" (id 1) (at 217.17 60.9599 0)
-      (effects (font (size 1.27 1.27)) (justify right))
-    )
-    (property "Footprint" "Capacitor_SMD:C_0805_2012Metric" (id 2) (at 212.3948 55.88 0)
-      (effects (font (size 1.27 1.27)) hide)
-    )
-    (property "Datasheet" "https://datasheets.kyocera-avx.com/X7RDielectric.pdf" (id 3) (at 213.36 59.69 0)
+    (property "Value" "" (id 1) (at 217.17 60.9599 0)
+      (effects (font (size 1.27 1.27)) (justify right))
+    )
+    (property "Footprint" "" (id 2) (at 212.3948 55.88 0)
+      (effects (font (size 1.27 1.27)) hide)
+    )
+    (property "Datasheet" "https://search.murata.co.jp/Ceramy/image/img/A01X/G101/ENG/GRM2195C1H512JA01-01.pdf" (id 3) (at 213.36 59.69 0)
       (effects (font (size 1.27 1.27)) hide)
     )
@@
       (effects (font (size 1.27 1.27)) (justify right))
     )
-    (property "Value" "5n" (id 1) (at 217.17 109.2199 0)
-      (effects (font (size 1.27 1.27)) (justify right))
-    )
-    (property "Footprint" "Capacitor_SMD:C_0805_2012Metric" (id 2) (at 212.3948 104.14 0)
-      (effects (font (size 1.27 1.27)) hide)
-    )
-    (property "Datasheet" "https://datasheets.kyocera-avx.com/X7RDielectric.pdf" (id 3) (at 213.36 107.95 0)
+    (property "Value" "" (id 1) (at 217.17 109.2199 0)
+      (effects (font (size 1.27 1.27)) (justify right))
+    )
+    (property "Footprint" "" (id 2) (at 212.3948 104.14 0)
+      (effects (font (size 1.27 1.27)) hide)
+    )
+    (property "Datasheet" "https://search.murata.co.jp/Ceramy/image/img/A01X/G101/ENG/GRM2195C1H512JA01-01.pdf" (id 3) (at 213.36 107.95 0)
       (effects (font (size 1.27 1.27)) hide)
     )
@@
     (in_bom yes) (on_board yes)
     (property "Reference" "R8" (id 0) (at 254 74.93 90))
-    (property "Value" "22k" (id 1) (at 255.27 77.47 90))
-    (property "Footprint" "Resistor_SMD:R_0805_2012Metric" (id 2) (at 250.19 81.788 90)
-      (effects (font (size 1.27 1.27)) hide)
-    )
-    (property "Datasheet" "https://www.meritekusa.com/wp-content/uploads/2018/06/Standard-Chip-Resistor-CR-Series.pdf" (id 3) (at 250.19 80.01 0)
-      (effects (font (size 1.27 1.27)) hide)
-    )
+    (property "Value" "" (id 1) (at 255.27 77.47 90))
+    (property "Footprint" "" (id 2) (at 250.19 81.788 90)
+      (effects (font (size 1.27 1.27)) hide)
+    )
+    (property "Datasheet" "https://www.te.com/commerce/DocumentDelivery/DDEController?Action=srchrtrv&DocNm=1773204&DocType=DS&DocLang=English" (id 3) (at 250.19 80.01 0)
+      (effects (font (size 1.27 1.27)) hide)
+    )
