File: Schematic/SDRrecV5/Complete Schematic V4.kicad_sch (KiCad schematic)
At the start: 73 parts, among them J1 Conn_Coaxial, J2 SJ1-3525N, U1 Si5351A-B-GT, U2 SN74CBT3253, U3 LT6231, U4 LM4562MA, Y1 Crystal_GND24_Small

Commit message: new changes to orgnization
Parts:
- C10, C11, C12, C9: value (none) -> 5n; footprint (none) -> Capacitor_SMD:C_0805_2012Metric
- R8, R9: value (none) -> 22k; footprint (none) -> Resistor_SMD:R_0805_2012Metric
Connections:
- net GND: now also J1.2 (Ext); no longer J1.1 (In)
- net at C1.2, TP1.1: now also J1.1 (In); no longer J1.2 (Ext)
- net at C10.2, R5.1, TP4.1: now also U2.12 (2B3), U2.4 (1B3); no longer U2.11 (2B2), U2.5 (1B2)
- net at R14.1, R16.1: now also U4.2 (-); no longer U4.3 (+)
- net at C11.1, R6.1, TP5.1: now also U2.11 (2B2), U2.5 (1B2); no longer U2.12 (2B3), U2.4 (1B3)
- net at C22.1, R12.1: now also U4.3 (+); no longer U4.2 (-)
Other:
- moved on the sheet: J1
Changed lines of the file:
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@@
   (junction (at 336.55 180.34) (diameter 0) (color 0 0 0 0)
   )
+  (junction (at 266.7 24.13) (diameter 0) (color 0 0 0 0)
+  )
+  (junction (at 346.71 80.01) (diameter 0) (color 0 0 0 0)
+  )
+  (junction (at 271.78 66.04) (diameter 0) (color 0 0 0 0)
+  )
+  (junction (at 133.35 80.01) (diameter 0) (color 0 0 0 0)
+  )
+  (junction (at 260.35 101.6) (diameter 0) (color 0 0 0 0)
+  )
+  (junction (at 224.79 104.14) (diameter 0) (color 0 0 0 0)
+  )
+  (junction (at 365.76 43.18) (diameter 0) (color 0 0 0 0)
+  )
+  (junction (at 205.74 90.17) (diameter 0) (color 0 0 0 0)
+  )
+  (junction (at 271.78 101.6) (diameter 0) (color 0 0 0 0)
+  )
+  (junction (at 223.52 99.06) (diameter 0) (color 0 0 0 0)
+  )
+  (junction (at 209.55 189.23) (diameter 0) (color 0 0 0 0)
+  )
+  (junction (at 242.57 68.58) (diameter 0) (color 0 0 0 0)
+  )
+  (junction (at 172.72 59.69) (diameter 0) (color 0 0 0 0)
+  )
+  (junction (at 242.57 104.14) (diameter 0) (color 0 0 0 0)
+  )
+  (junction (at 285.75 88.9) (diameter 0) (color 0 0 0 0)
+  )
+  (junction (at 231.14 179.07) (diameter 0) (color 0 0 0 0)
+  )
   (junction (at 213.36 68.58) (diameter 0) (color 0 0 0 0)
   )
-  (junction (at 266.7 24.13) (diameter 0) (color 0 0 0 0)
-  )
-  (junction (at 346.71 80.01) (diameter 0) (color 0 0 0 0)
-  )
-  (junction (at 271.78 66.04) (diameter 0) (color 0 0 0 0)
-  )
-  (junction (at 133.35 80.01) (diameter 0) (color 0 0 0 0)
-  )
-  (junction (at 260.35 101.6) (diameter 0) (color 0 0 0 0)
-  )
-  (junction (at 224.79 104.14) (diameter 0) (color 0 0 0 0)
-  )
-  (junction (at 365.76 43.18) (diameter 0) (color 0 0 0 0)
-  )
-  (junction (at 271.78 101.6) (diameter 0) (color 0 0 0 0)
-  )
-  (junction (at 223.52 99.06) (diameter 0) (color 0 0 0 0)
-  )
-  (junction (at 209.55 189.23) (diameter 0) (color 0 0 0 0)
-  )
-  (junction (at 201.93 92.71) (diameter 0) (color 0 0 0 0)
-  )
-  (junction (at 242.57 68.58) (diameter 0) (color 0 0 0 0)
-  )
-  (junction (at 172.72 59.69) (diameter 0) (color 0 0 0 0)
-  )
-  (junction (at 242.57 104.14) (diameter 0) (color 0 0 0 0)
-  )
-  (junction (at 285.75 88.9) (diameter 0) (color 0 0 0 0)
-  )
-  (junction (at 231.14 179.07) (diameter 0) (color 0 0 0 0)
-  )
   (junction (at 335.28 80.01) (diameter 0) (color 0 0 0 0)
   )
@@
   (junction (at 209.55 181.61) (diameter 0) (color 0 0 0 0)
   )
-  (junction (at 205.74 77.47) (diameter 0) (color 0 0 0 0)
-  )
   (junction (at 213.36 104.14) (diameter 0) (color 0 0 0 0)
   )
@@
   )
   (junction (at 213.36 63.5) (diameter 0) (color 0 0 0 0)
+  )
+  (junction (at 201.93 80.01) (diameter 0) (color 0 0 0 0)
   )
   (junction (at 69.85 158.75) (diameter 0) (color 0 0 0 0)
@@
   (no_connect (at 287.02 156.21))
   (no_connect (at 287.02 173.99))
-  (wire (pts (xy 205.74 68.58) (xy 205.74 77.47))
-    (stroke (width 0) (type default) (color 0 0 0 0))
-  )
   (wire (pts (xy 308.61 138.43) (xy 308.61 137.16))
     (stroke (width 0) (type default) (color 0 0 0 0))
@@
     (stroke (width 0) (type default) (color 0 0 0 0))
   )
+  (wire (pts (xy 205.74 99.06) (xy 213.36 99.06))
+    (stroke (width 0) (type default) (color 0 0 0 0))
+  )
   (wire (pts (xy 133.35 62.23) (xy 133.35 66.04))
     (stroke (width 0) (type default) (color 0 0 0 0))
@@
     (stroke (width 0) (type default) (color 0 0 0 0))
   )
+  (wire (pts (xy 207.01 80.01) (xy 207.01 68.58))
+    (stroke (width 0) (type default) (color 0 0 0 0))
+  )
   (wire (pts (xy 133.35 95.25) (xy 133.35 93.98))
     (stroke (width 0) (type default) (color 0 0 0 0))
@@
     (stroke (width 0) (type default) (color 0 0 0 0))
   )
-  (wire (pts (xy 201.93 92.71) (xy 201.93 99.06))
-    (stroke (width 0) (type default) (color 0 0 0 0))
-  )
   (wire (pts (xy 105.41 80.01) (xy 110.49 80.01))
     (stroke (width 0) (type default) (color 0 0 0 0))
@@
     (stroke (width 0) (type default) (color 0 0 0 0))
   )
-  (wire (pts (xy 201.93 99.06) (xy 213.36 99.06))
+  (wire (pts (xy 205.74 90.17) (xy 205.74 99.06))
     (stroke (width 0) (type default) (color 0 0 0 0))
   )
@@
     (stroke (width 0) (type default) (color 0 0 0 0))
   )
-  (wire (pts (xy 205.74 68.58) (xy 213.36 68.58))
-    (stroke (width 0) (type default) (color 0 0 0 0))
-  )
   (wire (pts (xy 224.79 109.22) (xy 224.79 104.14))
     (stroke (width 0) (type default) (color 0 0 0 0))
@@
     (stroke (width 0) (type default) (color 0 0 0 0))
   )
+  (wire (pts (xy 207.01 68.58) (xy 213.36 68.58))
+    (stroke (width 0) (type default) (color 0 0 0 0))
+  )
   (wire (pts (xy 231.14 176.53) (xy 231.14 179.07))
     (stroke (width 0) (type default) (color 0 0 0 0))
@@
   )
   (wire (pts (xy 157.48 95.25) (xy 157.48 96.52))
+    (stroke (width 0) (type default) (color 0 0 0 0))
+  )
+  (wire (pts (xy 201.93 80.01) (xy 207.01 80.01))
     (stroke (width 0) (type default) (color 0 0 0 0))
   )
@@
     (in_bom yes) (on_board yes)
     (property "Reference" "R9" (id 0) (at 255.27 111.76 90))
-    (property "Value" "" (id 1) (at 255.27 114.3 90))
-    (property "Footprint" "" (id 2) (at 250.19 117.348 90)
+    (property "Value" "22k" (id 1) (at 255.27 114.3 90))
+    (property "Footprint" "Resistor_SMD:R_0805_2012Metric" (id 2) (at 250.19 117.348 90)
       (effects (font (size 1.27 1.27)) hide)
     )
@@
       (effects (font (size 1.27 1.27)) (justify right))
     )
-    (property "Value" "" (id 1) (at 217.17 73.6599 0)
-      (effects (font (size 1.27 1.27)) (justify right))
-    )
-    (property "Footprint" "" (id 2) (at 212.3948 68.58 0)
+    (property "Value" "5n" (id 1) (at 217.17 73.6599 0)
+      (effects (font (size 1.27 1.27)) (justify right))
+    )
+    (property "Footprint" "Capacitor_SMD:C_0805_2012Metric" (id 2) (at 212.3948 68.58 0)
       (effects (font (size 1.27 1.27)) hide)
     )
@@
       (effects (font (size 1.27 1.27)) (justify right))
     )
-    (property "Value" "" (id 1) (at 217.17 96.5199 0)
-      (effects (font (size 1.27 1.27)) (justify right))
-    )
-    (property "Footprint" "" (id 2) (at 212.3948 91.44 0)
+    (property "Value" "5n" (id 1) (at 217.17 96.5199 0)
+      (effects (font (size 1.27 1.27)) (justify right))
+    )
+    (property "Footprint" "Capacitor_SMD:C_0805_2012Metric" (id 2) (at 212.3948 91.44 0)
       (effects (font (size 1.27 1.27)) hide)
     )
@@
     (pin "1")
   )
-  (symbol (lib_id "lt6231:LT6231") (at 326.39 78.74 0) (unit 1)
+  (symbol (lib_id "lt6231:LT6231") (at 326.39 78.74 0) (mirror x) (unit 1)
     (in_bom yes) (on_board yes) (fields_autoplaced)
     (property "Reference" "U4" (id 0) (at 326.39 68.58 0))
@@
       (effects (font (size 1.27 1.27)) (justify right))
     )
-    (property "Value" "" (id 1) (at 217.17 60.9599 0)
-      (effects (font (size 1.27 1.27)) (justify right))
-    )
-    (property "Footprint" "" (id 2) (at 212.3948 55.88 0)
+    (property "Value" "5n" (id 1) (at 217.17 60.9599 0)
+      (effects (font (size 1.27 1.27)) (justify right))
+    )
+    (property "Footprint" "Capacitor_SMD:C_0805_2012Metric" (id 2) (at 212.3948 55.88 0)
       (effects (font (size 1.27 1.27)) hide)
     )
@@
     (pin "2")
   )
-  (symbol (lib_id "Connector:Conn_Coaxial") (at 45.72 80.01 90) (unit 1)
-    (in_bom yes) (on_board yes) (fields_autoplaced)
-    (property "Reference" "J1" (id 0) (at 46.0132 72.39 90))
-    (property "Value" "Conn_Coaxial" (id 1) (at 46.0132 74.93 90))
+  (symbol (lib_id "Connector:Conn_Coaxial") (at 45.72 80.01 0) (mirror y) (unit 1)
+    (in_bom yes) (on_board yes) (fields_autoplaced)
+    (property "Reference" "J1" (id 0) (at 46.0374 72.39 0))
+    (property "Value" "Conn_Coaxial" (id 1) (at 46.0374 74.93 0))
     (property "Footprint" "Connector_Coaxial:BNC_Amphenol_B6252HB-NPP3G-50_Horizontal" (id 2) (at 45.72 80.01 0)
       (effects (font (size 1.27 1.27)) hide)
@@
       (effects (font (size 1.27 1.27)) (justify right))
     )
-    (property "Value" "" (id 1) (at 217.17 109.2199 0)
-      (effects (font (size 1.27 1.27)) (justify right))
-    )
-    (property "Footprint" "" (id 2) (at 212.3948 104.14 0)
+    (property "Value" "5n" (id 1) (at 217.17 109.2199 0)
+      (effects (font (size 1.27 1.27)) (justify right))
+    )
+    (property "Footprint" "Capacitor_SMD:C_0805_2012Metric" (id 2) (at 212.3948 104.14 0)
       (effects (font (size 1.27 1.27)) hide)
     )
@@
     (in_bom yes) (on_board yes)
     (property "Reference" "R8" (id 0) (at 254 74.93 90))
-    (property "Value" "" (id 1) (at 255.27 77.47 90))
-    (property "Footprint" "" (id 2) (at 250.19 81.788 90)
-      (effects (font (size 1.27 1.27)) hide)
-    )
+    (property "Value" "22k" (id 1) (at 255.27 77.47 90))
+    (property "Footprint" "Resistor_SMD:R_0805_2012Metric" (id 2) (at 250.19 81.788 90)
+      (effects (font (size 1.27 1.27)) hide)
+    )
