File: Schematic Files/SDRrecV5/KiCAD Files/Complete Schematic V5.kicad_sch (KiCad schematic)
At the start: 73 parts, among them J1 Conn_Coaxial, J2 SJ1-3525N, U1 Si5351A-B-GT, U2 SN74CBT3253, U3 LT6231, U4 LM4562MA, Y1 Crystal_GND24_Small

Commit message: Created New Folders
Parts:
- removed C18: 0.1u, Capacitor_SMD:C_0805_2012Metric, symbol Device:C
- removed C19, C20, C22, C23: 100p, Capacitor_SMD:C_0805_2012Metric, symbol Device:C
- removed R10, R11: 4.64k, Resistor_SMD:R_0805_2012Metric, symbol Device:R
- removed R12, R13: 52.3k, Resistor_SMD:R_0805_2012Metric, symbol Device:R
- removed R14, R15: 2.49k, Resistor_SMD:R_0805_2012Metric, symbol Device:R
- removed R16, R17: 17.4k, Resistor_SMD:R_0805_2012Metric, symbol Device:R
- removed TP10, TP9: TestPoint, TestPoint:TestPoint_THTPad_2.0x2.0mm_Drill1.0mm, symbol Connector:TestPoint
- removed U4: LM4562MA, Package_SO:SOIC-8_3.9x4.9mm_P1.27mm, symbol lt6231:LT6231
- added TP16: TestPoint, TestPoint:TestPoint_THTPad_2.0x2.0mm_Drill1.0mm, symbol Connector:TestPoint
- C13: value (none) -> 8200u; footprint (none) -> Capacitor_THT:CP_Radial_D16.0mm_P7.50mm
- R2, R3: footprint Resistor_SMD:R_2512_6332Metric -> Resistor_SMD:R_0805_2012Metric
Connections:
- net GND: now also TP16.1
- net at C17.1, R9.2, TP8.1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: now also C27.2
- net at C16.1, R8.2, TP7.1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: now also C26.2
- net at C10.2, R5.1, TP4.1: now also U2.13 (2B4), U2.3 (1B4); no longer U2.12 (2B3), U2.4 (1B3)
- net at C12.2, R7.1, TP6.1: now also U2.12 (2B3), U2.4 (1B3); no longer U2.13 (2B4), U2.3 (1B4)
Other:
- moved on the sheet: C26, C27, J2, R20, R21, TP11, TP12
