File: Schematic Files/SDRrecV6/Complete Schematic V6.kicad_sch (KiCad schematic)
At the start: 58 parts, among them J1 Conn_Coaxial, J2 SJ1-3525N, U1 Si5351A-B-GT, U2 SN74CBT3253, U3 LT6231, Y1 Crystal_GND24_Small

Commit message: Updated V6 Board
Parts:
- J2: footprint Audio Jack_Stereo 3:Jack_3.5mm_stereo_TRS_jack -> (none)
Changed lines of the file:
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@@
     (pin "1")
+  )
+  (symbol (lib_id "SJ1-3525N:SJ1-3525N") (at 313.69 85.09 0) (mirror y) (unit 1)
+    (in_bom yes) (on_board yes) (fields_autoplaced)
+    (property "Reference" "J2" (id 0) (at 325.12 83.8199 0)
+      (effects (font (size 1.27 1.27)) (justify right))
+    )
+    (property "Value" "SJ1-3525N" (id 1) (at 325.12 86.3599 0)
+      (effects (font (size 1.27 1.27)) (justify right))
+    )
+    (property "Footprint" "" (id 2) (at 313.69 85.09 0)
+      (effects (font (size 1.27 1.27)) (justify left bottom) hide)
+    )
+    (property "Datasheet" "" (id 3) (at 313.69 85.09 0)
+      (effects (font (size 1.27 1.27)) (justify left bottom) hide)
+    )
+    (property "STANDARD" "Manufacturer recommendation" (id 4) (at 313.69 85.09 0)
+      (effects (font (size 1.27 1.27)) (justify left bottom) hide)
+    )
+    (property "MANUFACTURER" "CUI" (id 5) (at 313.69 85.09 0)
+      (effects (font (size 1.27 1.27)) (justify left bottom) hide)
+    )
+    (property "PARTREV" "1.02" (id 6) (at 313.69 85.09 0)
+      (effects (font (size 1.27 1.27)) (justify left bottom) hide)
+    )
+    (pin "1")
+    (pin "10")
+    (pin "11")
+    (pin "2")
+    (pin "3")
   )
   (symbol (lib_id "lt6231:LT6231") (at 231.14 43.18 270) (unit 3)
@@
     (pin "9")
   )
-  (symbol (lib_id "SJ1-3525N:SJ1-3525N") (at 313.69 85.09 0) (mirror y) (unit 1)
-    (in_bom yes) (on_board yes) (fields_autoplaced)
-    (property "Reference" "J2" (id 0) (at 325.12 83.8199 0)
-      (effects (font (size 1.27 1.27)) (justify right))
-    )
-    (property "Value" "SJ1-3525N" (id 1) (at 325.12 86.3599 0)
-      (effects (font (size 1.27 1.27)) (justify right))
-    )
-    (property "Footprint" "Audio Jack_Stereo 3:Jack_3.5mm_stereo_TRS_jack" (id 2) (at 313.69 85.09 0)
-      (effects (font (size 1.27 1.27)) (justify left bottom) hide)
-    )
-    (property "Datasheet" "https://www.cuidevices.com/product/resource/sj1-352xn.pdf" (id 3) (at 313.69 85.09 0)
-      (effects (font (size 1.27 1.27)) (justify left bottom) hide)
-    )
-    (property "STANDARD" "Manufacturer recommendation" (id 4) (at 313.69 85.09 0)
-      (effects (font (size 1.27 1.27)) (justify left bottom) hide)
-    )
-    (property "MANUFACTURER" "CUI" (id 5) (at 313.69 85.09 0)
-      (effects (font (size 1.27 1.27)) (justify left bottom) hide)
-    )
-    (property "PARTREV" "1.02" (id 6) (at 313.69 85.09 0)
-      (effects (font (size 1.27 1.27)) (justify left bottom) hide)
-    )
-    (pin "1")
-    (pin "10")
-    (pin "11")
-    (pin "2")
-    (pin "3")
-  )
   (symbol (lib_id "Device:C") (at 312.42 138.43 270) (unit 1)
     (in_bom yes) (on_board yes) (fields_autoplaced)
@@
       (reference "J1") (unit 1) (value "Conn_Coaxial") (footprint "Connector_Coaxial:BNC_Amphenol_B6252HB-NPP3G-50_Horizontal")
     )
-    (path "/e5b6d70d-eb40-43bd-afb8-b2b168a19d8c"
-      (reference "J2") (unit 1) (value "SJ1-3525N") (footprint "Audio Jack_Stereo 3:Jack_3.5mm_stereo_TRS_jack")
+    (path "/3aa5dba9-698a-429b-b5bc-746b0a7330f7"
+      (reference "J2") (unit 1) (value "SJ1-3525N") (footprint "CUI_SJ1-3225N:CUI_SJ1-3525N")
     )
     (path "/7492b8d4-527b-4a70-84f8-f67406097c5b"
