File: Schematic Files/Circuit Segment Schematics/BandPass Filter.kicad_sch (KiCad schematic)
At the start: 8 parts

Commit message: Created New Folders
Parts:
- added C4: (no value), symbol Device:C
- added R2, R3: (no value), symbol Device:R
- C1, C3: renamed from C?; value 220p -> (none)
- C2: renamed from C?; value 620p -> (none)
- L1, L3: renamed from L?; value 820n -> (none)
- L2: renamed from L?; value 720n -> (none)
- gave numbers to parts that had none: 2
Connections:
- net GND: now also J1.2 (Ext), C4.1, R3.2; no longer J1.1 (In)
- net at R1.1: now also J1.1 (In); no longer J1.2 (Ext)
- net Input to 1A and 2A on SN74CBT3253: now reaches L3.2
- net Input to 1A and 2A on SN74CBT3253: now also R2.2, R3.1
- new net Filtered 5V: C4.2, R2.1
Other:
- moved on the sheet: J1, L3

Commit message: Addel Gerber, PDF, and Drill Files. Addes Pictures Folder
Parts:
- C1, C3: value (none) -> 270p
- C2: value (none) -> 560p
- C4: value (none) -> 0.1u
- L2: value (none) -> 360n
- L3: value (none) -> 750n
- R2, R3: value (none) -> 10k
Changed lines of the file:
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@@
     (in_bom yes) (on_board yes) (fields_autoplaced)
     (property "Reference" "C1" (id 0) (at 118.11 78.74 90))
-    (property "Value" "" (id 1) (at 118.11 81.28 90))
+    (property "Value" "270p" (id 1) (at 118.11 81.28 90))
     (property "Footprint" "" (id 2) (at 114.3 87.3252 0)
       (effects (font (size 1.27 1.27)) hide)
@@
       (effects (font (size 1.27 1.27)) (justify left))
     )
-    (property "Value" "" (id 1) (at 175.26 80.0099 0)
+    (property "Value" "10k" (id 1) (at 175.26 80.0099 0)
       (effects (font (size 1.27 1.27)) (justify left))
     )
@@
       (effects (font (size 1.27 1.27)) (justify left))
     )
-    (property "Value" "" (id 1) (at 146.05 95.2499 0)
+    (property "Value" "360n" (id 1) (at 146.05 95.2499 0)
       (effects (font (size 1.27 1.27)) (justify left))
     )
@@
     (in_bom yes) (on_board yes) (fields_autoplaced)
     (property "Reference" "C4" (id 0) (at 168.91 62.23 90))
-    (property "Value" "" (id 1) (at 168.91 64.77 90))
+    (property "Value" "0.1u" (id 1) (at 168.91 64.77 90))
     (property "Footprint" "" (id 2) (at 172.72 68.8848 0)
       (effects (font (size 1.27 1.27)) hide)
@@
     (in_bom yes) (on_board yes) (fields_autoplaced)
     (property "Reference" "C3" (id 0) (at 153.67 78.74 90))
-    (property "Value" "" (id 1) (at 153.67 81.28 90))
+    (property "Value" "270p" (id 1) (at 153.67 81.28 90))
     (property "Footprint" "" (id 2) (at 157.48 85.3948 0)
       (effects (font (size 1.27 1.27)) hide)
@@
       (effects (font (size 1.27 1.27)) (justify left))
     )
-    (property "Value" "" (id 1) (at 175.26 95.2499 0)
+    (property "Value" "10k" (id 1) (at 175.26 95.2499 0)
       (effects (font (size 1.27 1.27)) (justify left))
     )
@@
       (effects (font (size 1.27 1.27)) (justify left))
     )
-    (property "Value" "" (id 1) (at 138.43 95.2499 0)
+    (property "Value" "560p" (id 1) (at 138.43 95.2499 0)
       (effects (font (size 1.27 1.27)) (justify left))
     )
@@
     (in_bom yes) (on_board yes) (fields_autoplaced)
     (property "Reference" "L3" (id 0) (at 163.83 80.01 90))
-    (property "Value" "" (id 1) (at 163.83 82.55 90))
+    (property "Value" "750n" (id 1) (at 163.83 82.55 90))
     (property "Footprint" "" (id 2) (at 163.83 86.36 0)
       (effects (font (size 1.27 1.27)) hide)
@@
       (effects (font (size 1.27 1.27)) hide)
     )
-    (property "Value" "" (id 1) (at 161.29 69.8499 90)
+    (property "Value" "GND" (id 1) (at 161.29 69.8499 90)
       (effects (font (size 1.27 1.27)) (justify right))
     )
@@
     )
     (path "/61d94937-c6a5-45c6-96c0-c3d70fb342d4"
-      (reference "L1") (unit 1) (value "270n") (footprint "")
+      (reference "L1") (unit 1) (value "750n") (footprint "")
     )
     (path "/428dc4cb-6b19-4973-91ed-389ce63058cf"
