File: Schematic Files/Circuit Segment Schematics/Arduino and Si5354.kicad_sch (KiCad schematic)
At the start: 10 parts, among them U1 Si5351A-B-GT, Y1 Crystal_GND24_Small

Commit message: Merge branch 'main' of https://github.com/cwill713/Software-Defined-Radio into Christian_V4
# Conflicts:
#	Schematic Files/Complete Schematic V4/Complete Schematic V4-backups/Complete Schematic V4-2022-04-28_000705.zip
#	Schematic Files/Complete Schematic V4/Complete Schematic V4-backups/Complete Schematic V4-2022-04-28_035923.zip
#	Schematic Files/Complete Schematic V4/Complete Schematic V4-backups/Complete Schematic V4-2022-04-28_040923.zip
#	Schematic Files/Complete Schematic V4/Complete Schematic V4-backups/Complete Schematic V4-2022-04-28_041923.zip
#	Schematic Files/Complete Schematic V4/Complete Schematic V4-backups/Complete Schematic V4-2022-04-28_042923.zip
#	Schematic Files/Complete Schematic V4/Complete Schematic V4-backups/Complete Schematic V4-2022-04-28_044216.zip
#	Schematic Files/Complete Schematic V4/Complete Schematic V4-backups/Complete Schematic V4-2022-04-28_045216.zip
#	Schematic Files/Complete Schematic V4/Complete Schematic V4.csv
#	Schematic Files/Complete Schematic V4/Complete Schematic V4.xlsx
#	Schematic Files/Complete Schematic V4/Complete Schematic V4.xml
#	Schematic Files/Complete Schematic V4/fp-lib-table
Connections:
- net CLK1 Output to S0 on SN74CBT3253 renamed CLK1 Output to S1 on SN74CBT3253
Changed lines of the file:
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@@
     (effects (font (size 1.27 1.27)) (justify right bottom))
   )
-  (label "CLK1 Output to S0 on SN74CBT3253" (at 125.73 114.3 0)
+  (label "CLK1 Output to S1 on SN74CBT3253" (at 125.73 114.3 0)
     (effects (font (size 1.27 1.27)) (justify left bottom))
   )
@@
       (effects (font (size 1.27 1.27)) hide)
     )
-    (property "Value" "" (id 1) (at 193.04 138.43 0))
+    (property "Value" "GND" (id 1) (at 193.04 138.43 0))
     (property "Footprint" "" (id 2) (at 194.31 133.35 0)
       (effects (font (size 1.27 1.27)) hide)
